File: pcb/Cruiser.sch (KiCad schematic (older format))
At the start: 46 parts, among them J1 USB-A, P1 BDM, P2 GND-T0-T1-T2-T3, SW1 Load, SW2 Reset, SW3 SOLDER_BRIDGE, SW4 SOLDER_BRIDGE, SW5 SOLDER_BRIDGE, U1 FT232RL, U2 MC9S12XDP512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

Commit message: Added Port AN0-8 header, Port T4-7 header and added Port A7 header.
Parts:
- added A7: PA7, symbol CONN_1
- added J2: USB_B-MICRO, symbol USB_B-MICRO
- added P3: A/D, symbol CONN_4X2
- added P4: T4-T5-T6-T7, symbol CONN_2X2
Connections:
- net labels added: AN0, AN1, AN2, AN3, AN4, AN5, AN6, AN7, PT4, PT5, PT6, PT7
- net labels removed: 5v-USB, USB-GND
- wire segments 111 -> 112
- no-connect marks 97 -> 85
Other:
- moved on the sheet: C10, D1, R6, R8

Commit message: Added solder bridge connections to allow the USB/CPU/VRH 5v lines to be separated on the schematic.
Parts:
- added P5: VRH, symbol CONN_1
- added P6: CPU-5v, symbol CONN_1
- added SW6, SW7: SOLDER_BRIDGE, symbol SOLDER_BRIDGE
Connections:
- net labels added: 5vdc-usb
- wire segments 112 -> 125
Changed lines of the file:
@@
 	8850 800  8850 1300
 Wire Wire Line
-	7750 800  8850 800
+	7750 800  8900 800
 Connection ~ 7750 1300
 Connection ~ 7750 800
@@
 	1    0    0    -1
 $EndComp
-Text GLabel 6000 2800 2    40   Input ~ 0
+Text GLabel 6450 2800 2    40   Input ~ 0
 5vdc-cpu
 Text Notes 7250 4450 1    40   ~ 0
@@
 X7R Ceramic
 Text GLabel 7750 800  0    40   Input ~ 0
-5vdc-cpu
+5vdc-usb
 Text GLabel 4900 1250 0    40   Input ~ 0
 5vdc-cpu
@@
 Text GLabel 6000 1700 2    20   Input ~ 0
 PCB-GND
-Text GLabel 6000 2700 2    40   Input ~ 0
-5vdc-cpu
 Text GLabel 7800 4000 2    40   Input ~ 0
 5vdc-cpu
@@
 PCB-GND
 Text GLabel 10950 750  0    40   Input ~ 0
-5vdc-cpu
+5vdc-usb
 Text GLabel 10450 3350 0    40   Input ~ 0
-5vdc-cpu
+5vdc-usb
 Connection ~ 10450 4600
 Text GLabel 6000 4400 2    40   Input ~ 0
@@
 $EndComp
 Connection ~ 6000 4700
+$Comp
+L SOLDER_BRIDGE SW7
+U 1 1 553E24FD
+P 9100 800
+F 0 "SW7" V 9200 800 50  0000 C CNN
+F 1 "SOLDER_BRIDGE" V 9000 800 40  0000 C CNN
+F 2 "" H 9100 800 60  0001 C CNN
+F 3 "" H 9100 800 60  0001 C CNN
+	1    9100 800
+	0    -1   -1   0
+$EndComp
+Text GLabel 9400 800  2    40   Input ~ 0
+5vdc-cpu
+Connection ~ 8850 800
+Connection ~ 8900 800
+Connection ~ 9300 800
+$Comp
+L SOLDER_BRIDGE SW6
+U 1 1 553E294D
+P 6250 2600
+F 0 "SW6" V 6350 2600 50  0000 C CNN
+F 1 "SOLDER_BRIDGE" V 6150 2600 40  0000 C CNN
+F 2 "" H 6250 2600 60  0001 C CNN
+F 3 "" H 6250 2600 60  0001 C CNN
+	1    6250 2600
+	-1   0    0    1
+$EndComp
+Wire Wire Line
+	6450 2800 6400 2800
+Wire Wire Line
+	6400 2800 6400 2850
+Wire Wire Line
+	6400 2850 6250 2850
+Wire Wire Line
+	6250 2850 6250 2800
+Wire Wire Line
+	6250 2800 6000 2800
+Wire Wire Line
+	6000 2700 6100 2700
+Wire Wire Line
+	6100 2700 6100 2400
+Wire Wire Line
+	6100 2400 6250 2400
+Wire Wire Line
+	6250 2400 6250 2350
+Wire Wire Line
+	6250 2350 6450 2350
+$Comp
+L CONN_1 P5
+U 1 1 553E2E31
+P 6600 2350
+F 0 "P5" H 6680 2350 40  0000 L CNN
+F 1 "VRH" H 6600 2405 30  0001 C CNN
+F 2 "" H 6600 2350 60  0001 C CNN
+F 3 "" H 6600 2350 60  0001 C CNN
+	1    6600 2350
+	1    0    0    -1
+$EndComp
+$Comp
+L CONN_1 P6
+U 1 1 553E2E75
+P 9550 700
+F 0 "P6" H 9630 700 40  0000 L CNN
+F 1 "CPU-5v" H 9550 755 30  0001 C CNN
+F 2 "" H 9550 700 60  0001 C CNN
+F 3 "" H 9550 700 60  0001 C CNN
+	1    9550 700
+	1    0    0    -1
+$EndComp
+Wire Wire Line
+	9400 700  9300 700
+Wire Wire Line
+	9300 700  9300 800
+Wire Wire Line
+	9300 800  9400 800
 $EndSCHEMATC

Commit message: Removed PT0-3 current limiting resistors, increase PCB length from 44.44mm to 50mm, added PK4 and PA7 pins, split USB-5v and CPU-5v which can be tied together with a solder bridge, added CPU-5v and VRH pins with a solder bridge to tie them together.
Parts:
- removed A7: PA7, symbol CONN_1
- removed P2: GND-T0-T1-T2-T3, symbol CONN_5
- removed P4: T4-T5-T6-T7, symbol CONN_2X2
- removed R13, R14, R15, R16: 1k, symbol R
- added P2: Port T, symbol CONN_4X2
- added P4: PA7-GND, symbol CONN_2
- added PK4: PK4, symbol CONN_1
Connections:
- net labels added: PA7, PT0, PT1, PT2, PT3
- wire segments 125 -> 103
- no-connect marks 85 -> 84
Changed lines of the file:
@@
 Connection ~ 10950 750
 Connection ~ 10950 1250
-Connection ~ 1050 2200
-Connection ~ 950  2200
-Connection ~ 850  2200
-Connection ~ 750  2200
-Wire Wire Line
-	750  2200 750  2500
-Wire Wire Line
-	750  2500 600  2500
-Wire Wire Line
-	600  2500 600  3000
-Wire Wire Line
-	600  3000 650  3000
-Wire Wire Line
-	650  3000 650  3300
-Wire Wire Line
-	950  2200 950  2650
-Wire Wire Line
-	950  2650 900  2650
-Wire Wire Line
-	900  2650 900  3200
-Connection ~ 1050 2650
-Connection ~ 900  3200
-Connection ~ 1050 3150
 Connection ~ 1200 3600
 Connection ~ 1200 3700
-Connection ~ 900  3700
-Connection ~ 650  3800
-Wire Wire Line
-	1050 3150 1050 3600
-Wire Wire Line
-	1050 3600 1200 3600
-Connection ~ 750  2650
-Connection ~ 750  3150
-Wire Wire Line
-	750  3750 1100 3750
-Wire Wire Line
-	750  3750 750  3150
-Wire Wire Line
-	650  3800 1050 3800
-Wire Wire Line
-	1050 3800 1050 3900
-Wire Wire Line
-	1050 3900 1200 3900
 Wire Notes Line
 	11100 5650 11100 6850
@@
 Connection ~ 8450 1200
 Connection ~ 8050 1200
-Wire Wire Line
-	1200 3800 1100 3800
-Wire Wire Line
-	1100 3800 1100 3750
 Connection ~ 1200 3800
 Connection ~ 1200 3900
-Connection ~ 650  3300
-Wire Wire Line
-	1200 3700 900  3700
-Wire Wire Line
-	1050 2650 1050 2200
-Wire Wire Line
-	750  2650 750  2600
-Wire Wire Line
-	750  2600 850  2600
-Wire Wire Line
-	850  2600 850  2200
 Wire Wire Line
 	1150 2200 1150 2300
-Connection ~ 1150 2200
 Connection ~ 1150 2250
 Wire Wire Line
@@
 	1    1150 2300
 	1    0    0    -1
-$EndComp
-$Comp
-L CONN_5 P2
-U 1 1 50D20649
-P 950 1800
-F 0 "P2" V 900 1800 50  0000 C CNN
-F 1 "GND-T0-T1-T2-T3" V 1000 1800 50  0000 C CNN
-F 2 "" H 950 1800 60  0001 C CNN
-F 3 "" H 950 1800 60  0001 C CNN
-	1    950  1800
-	0    1    -1   0
-$EndComp
-$Comp
-L R R16
-U 1 1 50A13AA3
-P 1050 2900
-F 0 "R16" V 1130 2900 50  0000 C CNN
-F 1 "1k" V 1050 2900 50  0000 C CNN
-F 2 "" H 1050 2900 60  0001 C CNN
-F 3 "" H 1050 2900 60  0001 C CNN
-	1    1050 2900
-	-1   0    0    1
-$EndComp
-$Comp
-L R R15
-U 1 1 50A13A42
-P 900 3450
-F 0 "R15" V 980 3450 50  0000 C CNN
-F 1 "1k" V 900 3450 50  0000 C CNN
-F 2 "" H 900 3450 60  0001 C CNN
-F 3 "" H 900 3450 60  0001 C CNN
-	1    900  3450
-	-1   0    0    1
-$EndComp
-$Comp
-L R R13
-U 1 1 509BDA7F
-P 650 3550
-F 0 "R13" V 730 3550 50  0000 C CNN
-F 1 "1k" V 650 3550 50  0000 C CNN
-F 2 "" H 650 3550 60  0001 C CNN
-F 3 "" H 650 3550 60  0001 C CNN
-	1    650  3550
-	-1   0    0    1
-$EndComp
-$Comp
-L R R14
-U 1 1 509BDA70
-P 750 2900
-F 0 "R14" V 830 2900 50  0000 C CNN
-F 1 "1k" V 750 2900 50  0000 C CNN
-F 2 "" H 750 2900 60  0001 C CNN
-F 3 "" H 750 2900 60  0001 C CNN
-	1    750  2900
-	-1   0    0    1
 $EndComp
 Text GLabel 10450 4600 0    20   Input ~ 0
@@
 NoConn ~ 1200 5200
 NoConn ~ 1200 5100
-NoConn ~ 1200 4700
 NoConn ~ 1200 4600
 NoConn ~ 1200 3500
@@
 Connection ~ 7500 1850
 Connection ~ 7500 2950
-Text GLabel 8700 4600 0    40   Input ~ 0
-PT4
-Text GLabel 9500 4600 2    40   Input ~ 0
-PT5
-Text GLabel 8700 4700 0    40   Input ~ 0
-PT6
-Text GLabel 9500 4700 2    40   Input ~ 0
-PT7
 Text GLabel 1200 4200 0    40   Input ~ 0
 PT4
@@
 Connection ~ 1200 4400
 Connection ~ 1200 4500
-$Comp
-L CONN_2X2 P4
-U 1 1 553C1C3C
-P 9100 4650
-F 0 "P4" H 9100 4800 50  0000 C CNN
-F 1 "T4-T5-T6-T7" H 9110 4520 40  0000 C CNN
-F 2 "" H 9100 4650 60  0000 C CNN
-F 3 "" H 9100 4650 60  0000 C CNN
-	1    9100 4650
-	1    0    0    -1
-$EndComp
-Connection ~ 8700 4600
-Connection ~ 8700 4700
-Connection ~ 9500 4600
-Connection ~ 9500 4700
-$Comp
-L CONN_1 A7
-U 1 1 553E1BE1
-P 6150 4700
-F 0 "A7" H 6230 4700 40  0000 L CNN
-F 1 "PA7" H 6150 4755 30  0001 C CNN
-F 2 "" H 6150 4700 60  0001 C CNN
-F 3 "" H 6150 4700 60  0001 C CNN
-	1    6150 4700
-	1    0    0    -1
-$EndComp
 Connection ~ 6000 4700
 $Comp
@@
 Wire Wire Line
 	9300 800  9400 800
+$Comp
+L CONN_1 PK4
+U 1 1 553E3467
+P 1050 4700
+F 0 "PK4" H 1130 4700 40  0000 L CNN
+F 1 "PK4" H 1050 4755 30  0001 C CNN
+F 2 "" H 1050 4700 60  0001 C CNN
+F 3 "" H 1050 4700 60  0001 C CNN
+	1    1050 4700
+	-1   0    0    1
+$EndComp
+Connection ~ 1200 4700
+$Comp
+L CONN_4X2 P2
+U 1 1 553E3A5F
+P 10500 4000
+F 0 "P2" H 10500 4250 50  0000 C CNN
+F 1 "Port T" V 10500 4000 40  0000 C CNN
+F 2 "" H 10500 4000 60  0000 C CNN
+F 3 "" H 10500 4000 60  0000 C CNN
+	1    10500 4000
+	1    0    0    -1
+$EndComp
+Text GLabel 10100 3850 0    40   Input ~ 0
+PT0
+Text GLabel 10100 3950 0    40   Input ~ 0
+PT2
+Text GLabel 10100 4050 0    40   Input ~ 0
+PT4
+Text GLabel 10100 4150 0    40   Input ~ 0
+PT6
+Text GLabel 10900 3850 2    40   Input ~ 0
+PT1
+Text GLabel 10900 3950 2    40   Input ~ 0
+PT3
+Text GLabel 10900 4050 2    40   Input ~ 0
+PT5
+Text GLabel 10900 4150 2    40   Input ~ 0
+PT7
+Connection ~ 10100 3850
+Connection ~ 10100 3950
+Connection ~ 10100 4050
+Connection ~ 10100 4150
+Connection ~ 10900 4150
+Connection ~ 10900 4050
+Connection ~ 10900 3950
+Connection ~ 10900 3850
+Text GLabel 1200 3600 0    40   Input ~ 0
+PT0
+Text GLabel 1200 3700 0    40   Input ~ 0
+PT1
+Text GLabel 1200 3800 0    40   Input ~ 0
+PT2
+Text GLabel 1200 3900 0    40   Input ~ 0
+PT3
+Text GLabel 6000 4700 2    40   Input ~ 0
+PA7
+$Comp
+L CONN_2 P4
+U 1 1 553E4424
+P 9300 4700
+F 0 "P4" V 9250 4700 40  0000 C CNN
+F 1 "PA7-GND" V 9350 4700 40  0000 C CNN
+F 2 "" H 9300 4700 60  0001 C CNN
+F 3 "" H 9300 4700 60  0001 C CNN
+	1    9300 4700
+	1    0    0    1
+$EndComp
+Text GLabel 8950 4800 0    40   Input ~ 0
+PA7
+Text GLabel 8950 4600 0    20   Input ~ 0
+PCB-GND
+Connection ~ 8950 4600
+Connection ~ 8950 4800
 $EndSCHEMATC

Commit message: Added a 4 position 0.100" header for PK4  CPU-5v  PA7 and GND, reconnected the MCU VRH pin to the CPU 5v pin next to it as the Cruiser will only be used with a single power supply.
Parts:
- removed P4: PA7-GND, symbol CONN_2
- removed P5: VRH, symbol CONN_1
- removed P6: CPU-5v, symbol CONN_1
- removed PK4: PK4, symbol CONN_1
- removed SW6: SOLDER_BRIDGE, symbol SOLDER_BRIDGE
- added P5: PK4-CPU-5v-PA7, symbol CONN_4
Connections:
- net labels added: PK4
- wire segments 103 -> 94
Changed lines of the file:
@@
 Sheet 1 1
 Title "Cruiser Dev Board"
-Date "27 apr 2015"
+Date "30 apr 2015"
 Rev "0.3-alpha"
 Comp "Andy Goss"
@@
 	1    0    0    -1
 $EndComp
-Text GLabel 6450 2800 2    40   Input ~ 0
+Text GLabel 6100 2750 2    40   Input ~ 0
 5vdc-cpu
 Text Notes 7250 4450 1    40   ~ 0
@@
 Connection ~ 9500 4050
 Connection ~ 9500 4150
-Text GLabel 7500 2950 2    20   Input ~ 0
-PCB-GND
-Text GLabel 7500 1850 2    20   Input ~ 0
-PCB-GND
-Connection ~ 7500 1850
-Connection ~ 7500 2950
 Text GLabel 1200 4200 0    40   Input ~ 0
 PT4
@@
 Connection ~ 8900 800
 Connection ~ 9300 800
-$Comp
-L SOLDER_BRIDGE SW6
-U 1 1 553E294D
-P 6250 2600
-F 0 "SW6" V 6350 2600 50  0000 C CNN
-F 1 "SOLDER_BRIDGE" V 6150 2600 40  0000 C CNN
-F 2 "" H 6250 2600 60  0001 C CNN
-F 3 "" H 6250 2600 60  0001 C CNN
-	1    6250 2600
-	-1   0    0    1
-$EndComp
-Wire Wire Line
-	6450 2800 6400 2800
-Wire Wire Line
-	6400 2800 6400 2850
-Wire Wire Line
-	6400 2850 6250 2850
-Wire Wire Line
-	6250 2850 6250 2800
-Wire Wire Line
-	6250 2800 6000 2800
+Wire Wire Line
+	6100 2800 6000 2800
 Wire Wire Line
 	6000 2700 6100 2700
 Wire Wire Line
-	6100 2700 6100 2400
-Wire Wire Line
-	6100 2400 6250 2400
-Wire Wire Line
-	6250 2400 6250 2350
-Wire Wire Line
-	6250 2350 6450 2350
-$Comp
-L CONN_1 P5
-U 1 1 553E2E31
-P 6600 2350
-F 0 "P5" H 6680 2350 40  0000 L CNN
-F 1 "VRH" H 6600 2405 30  0001 C CNN
-F 2 "" H 6600 2350 60  0001 C CNN
-F 3 "" H 6600 2350 60  0001 C CNN
-	1    6600 2350
-	1    0    0    -1
-$EndComp
-$Comp
-L CONN_1 P6
-U 1 1 553E2E75
-P 9550 700
-F 0 "P6" H 9630 700 40  0000 L CNN
-F 1 "CPU-5v" H 9550 755 30  0001 C CNN
-F 2 "" H 9550 700 60  0001 C CNN
-F 3 "" H 9550 700 60  0001 C CNN
-	1    9550 700
-	1    0    0    -1
-$EndComp
-Wire Wire Line
-	9400 700  9300 700
-Wire Wire Line
-	9300 700  9300 800
-Wire Wire Line
 	9300 800  9400 800
-$Comp
-L CONN_1 PK4
-U 1 1 553E3467
-P 1050 4700
-F 0 "PK4" H 1130 4700 40  0000 L CNN
-F 1 "PK4" H 1050 4755 30  0001 C CNN
-F 2 "" H 1050 4700 60  0001 C CNN
-F 3 "" H 1050 4700 60  0001 C CNN
-	1    1050 4700
-	-1   0    0    1
-$EndComp
 Connection ~ 1200 4700
 $Comp
@@
 Text GLabel 6000 4700 2    40   Input ~ 0
 PA7
-$Comp
-L CONN_2 P4
-U 1 1 553E4424
-P 9300 4700
-F 0 "P4" V 9250 4700 40  0000 C CNN
-F 1 "PA7-GND" V 9350 4700 40  0000 C CNN
-F 2 "" H 9300 4700 60  0001 C CNN
-F 3 "" H 9300 4700 60  0001 C CNN
-	1    9300 4700
-	1    0    0    1
-$EndComp
-Text GLabel 8950 4800 0    40   Input ~ 0
+Text GLabel 9450 5300 0    40   Input ~ 0
 PA7
-Text GLabel 8950 4600 0    20   Input ~ 0
-PCB-GND
-Connection ~ 8950 4600
-Connection ~ 8950 4800
+Text GLabel 1200 4700 0    40   Input ~ 0
+PK4
+Connection ~ 4200 6750
+Connection ~ 9150 5950
+Connection ~ 9650 5950
+Connection ~ 9650 5750
+Connection ~ 10150 5950
+Connection ~ 10200 6700
+Connection ~ 9400 800
+Text GLabel 9450 5200 0    40   Input ~ 0
+5vdc-cpu
+Text GLabel 9450 5100 0    20   Input ~ 0
+PCB-GND
+Text GLabel 9450 5000 0    40   Input ~ 0
+PK4
+$Comp
+L CONN_4 P5
+U 1 1 553FA598
+P 9800 5150
+F 0 "P5" V 9750 5150 50  0000 C CNN
+F 1 "PK4-CPU-5v-PA7" H 9600 5400 50  0000 C CNN
+F 2 "" H 9800 5150 60  0000 C CNN
+F 3 "" H 9800 5150 60  0000 C CNN
+	1    9800 5150
+	1    0    0    -1
+$EndComp
+Connection ~ 9450 5000
+Connection ~ 9450 5100
+Connection ~ 9450 5200
+Connection ~ 9450 5300
+Wire Wire Line
+	6100 2700 6100 2800
+Connection ~ 6100 2750
 $EndSCHEMATC

Commit message: Added all of Port T pins, all of Port B pins, the first 8 Port AN (Analog input) pins and the first four pins of Port P (Port P0-3).  Also added CAN RX/TX pins and a block for Port K4, GND, CPU +5v and Port A7.  This should give access to the more interesting pins. :)
Parts:
- added P4: PWM, symbol CONN_4
- added P6: Port B, symbol CONN_4X2
- added P7: CAN, symbol CONN_2
Connections:
- net labels added: PB0, PB1, PB2, PB3, PB4, PB5, PB6, PB7, PP0, PP1, PP2, PP3, RX-CAN, TX-CAN
- no-connect marks 84 -> 70
Other:
- note added: "The board is powered completely\nby the USB port, so no external\npower supply is needed."
- note added: "This goal of this project is to\ndevelop a small portable\ndevelopment board you can\ncarry with you to develop\ncode against."
- note removed: "The board is powered completely by the USB port,\nso no external power supply is needed."
- note removed: "This goal of this project is to develop a small portable\ndevelopment board you can carry with you to develop\ncode against."
- moved on the sheet: C5, H1, P2, P3, P5
